File: ProjetKicadPCBOT/ProjetKicadPCBOT.kicad_pcb (KiCad board)
At the start: 4 copper layers, 80 x 60 mm, 58 parts, among them J1 TOF, J2 Conn_02x04_Odd_Even, J3 Conn_ST_STDC14, J4 Screw_Terminal_01x02, J5 Screw_Terminal_01x02, J6 USB_C_Receptacle_USB2.0_16P, J7 Conn_01x02, SW1 SW_Push, SW3 SW_Push, U1 LSM6DSOX, U2 STM32G431KBT6, U3 DRV8411APWPR, U4 BQ25896, U5 AP2112K-3.3

Commit message: Il reste 6 warning et il faut arranger les écritures
Parts:
- C1, C10, C12, C13, C14, C15, C16, C17, C18, C19, C2, C20, C3, C4, C5, C6, C7: footprint Capacitor_SMD:C_0603_1608Metric_Pad1.08x0.95mm_HandSolder -> Library_PCBOT:C_0603_1608Metric_Pad1.08x0.95mm_HandSolder
- C21: footprint Capacitor_SMD:CP_Elec_6.3x3 -> Library_PCBOT:CP_Elec_6.3x3
- C8, C9: footprint Capacitor_SMD:C_0603_1608Metric_Pad1.08x0.95mm_HandSolder -> Library_PCBOT:C_0603_1608Metric_Pad1.08x0.95mm_HandSolder; moved to B.Cu
- D1, D2: footprint LED_SMD:LED_0603_1608Metric_Pad1.05x0.95mm_HandSolder -> Library_PCBOT:LED_0603_1608Metric_Pad1.05x0.95mm_HandSolder
- H1, H2, H3, H4: footprint MountingHole:MountingHole_3.2mm_M3_DIN965_Pad -> Library_PCBOT:MountingHole_3.2mm_M3_DIN965_Pad
- J1: footprint Connector_PinHeader_2.54mm:PinHeader_1x06_P2.54mm_Vertical -> Library_PCBOT:PinHeader_1x06_P2.54mm_Vertical
- J2: footprint Connector_PinHeader_2.54mm:PinHeader_2x04_P2.54mm_Vertical_SMD -> Connector_PinSocket_2.54mm:PinSocket_2x04_P2.54mm_Vertical
- J3: footprint Connector_PinHeader_1.27mm:PinHeader_2x07_P1.27mm_Vertical_SMD -> Library_PCBOT:PinHeader_2x07_P1.27mm_Vertical_SMD
- J4, J5: footprint TerminalBlock_Phoenix:TerminalBlock_Phoenix_MKDS-1,5-2-5.08_1x02_P5.08mm_Horizontal -> Library_PCBOT:TerminalBlock_Phoenix_MKDS-1,5-2-5.08_1x02_P5.08mm_Horizontal
- J6: footprint Connector_USB:USB_C_Receptacle_GCT_USB4105-xx-A_16P_TopMnt_Horizontal -> Library_PCBOT:USB_C_Receptacle_GCT_USB4105-xx-A_16P_TopMnt_Horizontal
- J7: footprint Connector_JST:JST_PH_S2B-PH-K_1x02_P2.00mm_Horizontal -> Library_PCBOT:JST_PH_S2B-PH-K_1x02_P2.00mm_Horizontal
- JP1, JP2: footprint Jumper:SolderJumper-2_P1.3mm_Open_TrianglePad1.0x1.5mm -> Library_PCBOT:SolderJumper-2_P1.3mm_Open_TrianglePad1.0x1.5mm
- L1: footprint Inductor_SMD:L_0805_2012Metric_Pad1.05x1.20mm_HandSolder -> Library_PCBOT:L_0805_2012Metric_Pad1.05x1.20mm_HandSolder
- R1, R10, R11, R12, R13, R14, R15, R2, R3, R4, R5, R6, R7, R8, R9: footprint Resistor_SMD:R_0805_2012Metric_Pad1.20x1.40mm_HandSolder -> Library_PCBOT:R_0805_2012Metric_Pad1.20x1.40mm_HandSolder
- SW1: footprint Button_Switch_SMD:SW_Push_1P1T_NO_E-Switch_TL3301NxxxxxG -> Library_PCBOT:SW_Push_1P1T_NO_E-Switch_TL3301NxxxxxG
- SW3: footprint Button_Switch_SMD:SW_Push_1P1T_NO_E-Switch_TL3301NxxxxxG -> Library_PCBOT:SW_Push_1P1T_NO_E-Switch_TL3301NxxxxxG; moved to B.Cu
- U1: footprint Package_LGA:LGA-14_3x2.5mm_P0.5mm_LayoutBorder3x4y -> Library_PCBOT:LGA-14_3x2.5mm_P0.5mm_LayoutBorder3x4y
- U2: footprint Package_QFP:LQFP-32_7x7mm_P0.8mm -> Library_PCBOT:LQFP-32_7x7mm_P0.8mm
- U3: footprint Package_SO:HTSSOP-16-1EP_4.4x5mm_P0.65mm_EP3.4x5mm_Mask3x3mm_ThermalVias -> Library_PCBOT:HTSSOP-16-1EP_4.4x5mm_P0.65mm_EP3.4x5mm_Mask3x3mm_ThermalVias
- U4: footprint Package_DFN_QFN:Texas_RQM0029A_VQFN-29_4x4mm_P0.4mm -> Library_PCBOT:WQFN-24-1EP_4x4mm_P0.5mm_EP2.45x2.45mm_ThermalVias
- U5: footprint Package_TO_SOT_SMD:SOT-23-5 -> Library_PCBOT:SOT-23-5
- moved C8 139.1 mm to (180.2, 86.0), turned to 90 degrees
- moved C9 136.9 mm to (178.3, 86.0), turned to 90 degrees
- moved SW1 130.5 mm to (180.1, 78.6)
- moved C4 128.0 mm to (164.1, 98.7), turned to 180 degrees
- moved C5 126.7 mm to (164.1, 96.5)
- moved R9 122.0 mm to (143.5, 95.6)
- moved R6 115.8 mm to (130.2, 96.9)
- moved R7 115.7 mm to (130.2, 99.6)
- moved R14 115.5 mm to (142.6, 89.4), turned to 180 degrees
- moved R15 115.2 mm to (142.6, 91.7)
- moved C7 115.2 mm to (155.0, 90.1), turned to 180 degrees
- moved R13 113.9 mm to (139.2, 89.5), turned to 90 degrees
- moved JP1 113.4 mm to (143.5, 81.4), turned to 90 degrees
- moved D2 112.3 mm to (147.8, 84.5), turned to 180 degrees
- moved C6 112.0 mm to (150.4, 93.5), turned to 180 degrees
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Connections:
- C1 pad 2: 0 -> GND
- C10 pad 1: GND -> Net-(U3-VM)
- C10 pad 2: Net-(U3-VM) -> GND
- R6 pad 1: Net-(J6-CC1) -> GND
- R6 pad 2: GND -> Net-(J6-CC1)
- U4 pad 13: (no net) -> Net-(J7-Pin_1)
- U4 pad 20: (no net) -> Net-(U4-SW1)
- U4 pad 25: (no net) -> GND
Routing:
- net +3.3V: track 0.00 -> 142.1 mm, vias 0 -> 15
- net GND: track 0.00 -> 139.7 mm, vias 0 -> 52
- net CE: track 0.00 -> 95.6 mm
- net XST: track 0.00 -> 81.7 mm, vias 0 -> 1
- net SDA: track 0.00 -> 72.7 mm, vias 0 -> 2
- net SCL: track 0.00 -> 66.2 mm, vias 0 -> 4
- net GPIO1: track 0.00 -> 59.4 mm
- net Net-(J5-Pin_2): track 0.00 -> 58.2 mm, vias 0 -> 1
- net TIM1_CH1N: track 0.00 -> 50.4 mm, vias 0 -> 2
- net NRST: track 0.00 -> 47.5 mm, vias 0 -> 2
- net INT: track 0.00 -> 45.3 mm, vias 0 -> 2
- net VBAT_SYS: track 0.00 -> 44.6 mm
- net TIM1_CH1: track 0.00 -> 43.8 mm, vias 0 -> 2
- net Net-(J7-Pin_1): track 0.00 -> 40.4 mm, vias 0 -> 2
- net Net-(J5-Pin_1): track 0.00 -> 39.3 mm, vias 0 -> 1
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- added copper zone on In2.Cu, net +3.3V
- added copper zone on B.Cu, net GND
- added copper zone on F.Cu, net GND
- added copper zone on In1.Cu, net GND
- added copper zone on F.Cu, net SYS1
- removed copper zone on B.Cu, net (none)
- removed copper zone on F.Cu, net (none)
