File: ProjetKicadPCBOT/ProjetKicadPCBOT.kicad_sch (KiCad schematic)
At the start: 0 parts

Commit message: .
Other:
- title: PC BOT -> PCB BOT rahim 974
Changed lines of the file:
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@@
 	(paper "A4")
 	(title_block
-		(title "PC BOT")
+		(title "PCB BOT rahim 974")
+		(date "2026-02-07")
+		(rev "1.0")
 		(company "ENSEA")
 	)
