File: Kicad10/ProjetKicadPCBOTFinal10.kicad_pcb (KiCad board)
At the start: 4 copper layers, 80 x 60 mm, 58 parts, among them J1 TOF, J2 Conn_02x04_Odd_Even, J3 Conn_ST_STDC14, J4 Screw_Terminal_01x02, J5 Screw_Terminal_01x02, J6 USB_C_Receptacle_USB2.0_16P, J7 Conn_01x02, SW1 SW_Push, SW3 SW_Push, U1 LSM6DSOX, U2 STM32G431KBT6, U3 DRV8411APWPR, U4 BQ25896, U5 AP2112K-3.3

Commit message: Ajout final de la sérigraphie
Routing:
- net SPI1_MOSI: track 17.6 -> 16.7 mm
Other:
- board text added: "+"
- board text added: "-"
- board text added: "-- +3.3 SWDIO GND SWCLK GND - - - GND NRST UART_RX UART_TX"
- board text added: "AOUT1"
- board text added: "AOUT2"
- board text added: "BOUT1"
- board text added: "BOUT2"
- board text added: "GND"
- board text added: "GPIO1"
- board text added: "PC BOT 1 2026"
- board text added: "SCL"
- board text added: "SDA"
- board text added: "SPI1_MISO NRF_IRQ SPI1_SCK SPI1_MOSI NRF_CE NRF_CSN GND +3.3V"
- board text added: "XST"
Changed lines of the file:
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@@
 		(capping no)
 		(filling no)
-		(zone_defaults)
 		(pcbplotparams
 			(layerselection 0x00000000_00000000_55555555_5755f5ff)
@@
 			(usegerberattributes yes)
 			(usegerberadvancedattributes yes)
-			(creategerberjobfile yes)
+			(creategerberjobfile no)
 			(dashed_line_dash_ratio 12)
 			(dashed_line_gap_ratio 3)
@@
 			(outputformat 1)
 			(mirror no)
-			(drillshape 1)
+			(drillshape 0)
 			(scaleselection 1)
-			(outputdirectory "")
+			(outputdirectory "pcbot_gerber/")
 		)
 	)
@@
 		)
 		(fp_text user "${REFERENCE}"
-			(at 1 2.5 270)
+			(at 0.5 2 270)
 			(layer "F.Fab")
 			(effects
@@
 		(layer "Edge.Cuts")
 	)
+	(gr_text "+"
+		(at 124.12 72.32 0)
+		(layer "F.SilkS")
+		(effects
+			(font
+				(size 1 1)
+				(thickness 0.1)
+			)
+			(justify left bottom)
+		)
+	)
+	(gr_text "PC BOT 1 2026\n\n"
+		(at 125.97 124.64 0)
+		(layer "F.SilkS")
+		(effects
+			(font
+				(size 1 1)
+				(thickness 0.1)
+			)
+			(justify left bottom)
+		)
+	)
+	(gr_text "GPIO1"
+		(at 185.56 102.97 0)
+		(layer "F.SilkS")
+		(effects
+			(font
+				(size 1 1)
+				(thickness 0.1)
+			)
+			(justify left bottom)
+		)
+	)
+	(gr_text "GND"
+		(at 186.68 93.06 0)
+		(layer "F.SilkS")
+		(effects
+			(font
+				(size 1 1)
+				(thickness 0.1)
+			)
+			(justify left bottom)
+		)
+	)
+	(gr_text "SCL"
+		(at 186.83 97.5 0)
+		(layer "F.SilkS")
+		(effects
+			(font
+				(size 1 1)
+				(thickness 0.1)
+			)
+			(justify left bottom)
+		)
+	)
+	(gr_text "SDA"
+		(at 186.88 98.97 0)
+		(layer "F.SilkS")
+		(effects
+			(font
+				(size 1 1)
+				(thickness 0.1)
+			)
+			(justify left bottom)
+		)
+	)
+	(gr_text "XST"
+		(at 187.22 104.59 0)
+		(layer "F.SilkS")
+		(effects
+			(font
+				(size 1 1)
+				(thickness 0.1)
+			)
+			(justify left bottom)
+		)
+	)
+	(gr_text "-"
+		(at 125.26 75.28 90)
+		(layer "F.SilkS")
+		(effects
+			(font
+				(size 1 1)
+				(thickness 0.1)
+			)
+			(justify left bottom)
+		)
+	)
+	(gr_text "AOUT2"
+		(at 133.16 114.84 -0)
+		(layer "B.SilkS")
+		(effects
+			(font
+				(size 1 1)
+				(thickness 0.1)
+			)
+			(justify left bottom mirror)
+		)
+	)
+	(gr_text "AOUT1"
+		(at 141.18 114.88 -0)
+		(layer "B.SilkS")
+		(effects
+			(font
+				(size 1 1)
+				(thickness 0.1)
+			)
+			(justify left bottom mirror)
+		)
+	)
+	(gr_text "BOUT2"
+		(at 170.7 107.74 -0)
+		(layer "B.SilkS")
+		(effects
+			(font
+				(size 1 1)
+				(thickness 0.1)
+			)
+			(justify left bottom mirror)
+		)
+	)
+	(gr_text "SPI1_MISO NRF_IRQ\nSPI1_SCK SPI1_MOSI\nNRF_CE NRF_CSN\nGND +3.3V"
+		(at 172.54 75.43 -0)
+		(layer "B.SilkS")
+		(effects
+			(font
+				(size 1 1)
+				(thickness 0.1)
+			)
+			(justify left bottom mirror)
+		)
+	)
+	(gr_text "BOUT1"
+		(at 184.01 114.8 -0)
+		(layer "B.SilkS")
+		(effects
+			(font
+				(size 1 1)
+				(thickness 0.1)
+			)
+			(justify left bottom mirror)
+		)
+	)
+	(gr_text "--\n+3.3 SWDIO\nGND SWCLK\nGND -\n- -\nGND NRST\nUART_RX UART_TX"
+		(at 188.89 81.71 -0)
+		(layer "B.SilkS")
+		(effects
+			(font
+				(size 1 1)
+				(thickness 0.1)
+			)
+			(justify left bottom mirror)
+		)
+	)
 	(segment
 		(start 132.76 81.75)
@@
 	)
 	(segment
-		(start 153.373 88.083)
-		(end 153.373 77.48)
+		(start 153.373 78.237)
+		(end 154.11 77.5)
 		(width 0.2)
 		(layer "B.Cu")
@@
 	)
 	(segment
-		(start 153.373 77.48)
-		(end 153.393 77.5)
+		(start 154.11 77.5)
+		(end 157.46 77.5)
 		(width 0.2)
 		(layer "B.Cu")
@@
 	)
 	(segment
-		(start 153.393 77.5)
-		(end 157.46 77.5)
+		(start 153.373 88.083)
+		(end 153.373 78.237)
 		(width 0.2)
 		(layer "B.Cu")
@@
 	)
 	(segment
-		(start 154.204 82.58)
+		(start 154.644 82.58)
 		(end 157.46 82.58)
 		(width 0.2)
@@
 	(segment
 		(start 154.124 86.509026)
-		(end 154.124 82.5)
+		(end 154.124 83.1)
 		(width 0.2)
 		(layer "B.Cu")
@@
 	)
 	(segment
-		(start 154.124 82.5)
-		(end 154.204 82.58)
+		(start 154.124 83.1)
+		(end 154.644 82.58)
 		(width 0.2)
 		(layer "B.Cu")
@@
 	)
 	(segment
-		(start 157.6 90.48)
-		(end 153.774 86.654)
+		(start 153.774 80.836)
+		(end 154.57 80.04)
 		(width 0.2)
 		(layer "B.Cu")
@@
 	(segment
 		(start 153.774 86.654)
-		(end 153.774 79.756)
+		(end 153.774 80.836)
 		(width 0.2)
 		(layer "B.Cu")
@@
 	)
 	(segment
-		(start 153.774 79.756)
-		(end 154.058 80.04)
+		(start 154.57 80.04)
+		(end 157.46 80.04)
 		(width 0.2)
 		(layer "B.Cu")
@@
 	)
 	(segment
-		(start 154.058 80.04)
-		(end 157.46 80.04)
+		(start 157.6 90.48)
+		(end 153.774 86.654)
 		(width 0.2)
 		(layer "B.Cu")
