File: Kicad10/ProjetKicadPCBOTFinal.kicad_pcb (KiCad board)
At the start: 4 copper layers, 80 x 60 mm, 58 parts, among them J1 TOF, J2 Conn_02x04_Odd_Even, J3 Conn_ST_STDC14, J4 Screw_Terminal_01x02, J5 Screw_Terminal_01x02, J6 USB_C_Receptacle_USB2.0_16P, J7 Conn_01x02, SW1 SW_Push, SW3 SW_Push, U1 LSM6DSOX, U2 STM32G431KBT6, U3 DRV8411APWPR, U4 BQ25896, U5 AP2112K-3.3

Commit message: Update KiCad PCB et readme
Parts:
- C4: value 1010nF -> 10nF
Changed lines of the file:
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@@
 			)
 		)
-		(property "Value" "1010nF"
+		(property "Value" "10nF"
 			(at 0 1.43 180)
 			(layer "F.Fab")
